File: hardware/gps_tracker_basic.kicad_pcb (KiCad board)
At the start: 2 copper layers, 54 x 54 mm, 109 parts, among them J1 Conn_01x05, J2 USB_B_Micro, J3 Battery, J4 Conn_01x05, Q1 S8050, Q2 S8050, Q3 Si2301CDS, Q4 S8050, SW1 SW_Push_DPDT, SW2 SW_Push_DPDT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

Commit message: Update kicad sheets
Other:
- net class Default removed
