File: hardware/gps_tracker_basic.kicad_sch (KiCad schematic)
At the start: 65 parts, among them J1 Conn_01x05, J4 Conn_01x05, Q1 S8050, Q2 S8050, SW1 SW_Push_DPDT, SW2 SW_Push_DPDT, U1 STM32F030R8Tx, U2 CAT24C256, U3 FT230XS, U5 USBLC6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

Commit message: Update kicad sheets
Other:
- company: Ricardo Goncalves -> The Antenna Guy
Changed lines of the file:
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@@
     (date "2020-11-07")
     (rev "1.0")
-    (company "Ricardo Goncalves")
+    (company "The Antenna Guy")
   )
   (junction (at 140.97 184.15) (diameter 0) (color 0 0 0 0)
@@
     (pin "1")
   )
-  (symbol (lib_id "Device:R") (at 245.11 125.73 270)
+  (symbol (lib_id "Device:R") (at 245.11 125.73 270) (unit 1)
     (in_bom yes) (on_board yes)
     (property "Reference" "R17" (id 0) (at 245.11 123.19 90))
@@
     (pin "2")
   )
-  (symbol (lib_id "Device:R") (at 250.19 129.54 0)
+  (symbol (lib_id "Device:R") (at 250.19 129.54 0) (unit 1)
     (in_bom yes) (on_board yes)
     (property "Reference" "R19" (id 0) (at 251.46 129.54 0)
@@
     (pin "2")
   )
-  (symbol (lib_id "power:GND") (at 262.89 133.35 0)
+  (symbol (lib_id "power:GND") (at 262.89 133.35 0) (unit 1)
     (in_bom yes) (on_board yes)
     (property "Reference" "#PWR020" (id 0) (at 262.89 139.7 0)
@@
     (pin "1")
   )
-  (symbol (lib_id "Device:R") (at 262.89 114.3 0)
+  (symbol (lib_id "Device:R") (at 262.89 114.3 0) (unit 1)
     (in_bom yes) (on_board yes)
     (property "Reference" "R21" (id 0) (at 265.43 114.3 0))
@@
     (pin "2")
   )
-  (symbol (lib_id "Device:Q_NPN_BEC") (at 260.35 125.73 0)
+  (symbol (lib_id "Device:Q_NPN_BEC") (at 260.35 125.73 0) (unit 1)
     (in_bom yes) (on_board yes)
     (property "Reference" "Q1" (id 0) (at 265.2014 124.5616 0)
@@
     (pin "2")
   )
-  (symbol (lib_id "Device:R") (at 196.85 125.73 270)
+  (symbol (lib_id "Device:R") (at 196.85 125.73 270) (unit 1)
     (in_bom yes) (on_board yes)
     (property "Reference" "R18" (id 0) (at 196.85 123.19 90))
@@
     (pin "2")
   )
-  (symbol (lib_id "Device:R") (at 201.93 129.54 0)
+  (symbol (lib_id "Device:R") (at 201.93 129.54 0) (unit 1)
     (in_bom yes) (on_board yes)
     (property "Reference" "R20" (id 0) (at 203.2 129.54 0)
@@
     (pin "2")
   )
-  (symbol (lib_id "power:GND") (at 214.63 133.35 0)
+  (symbol (lib_id "power:GND") (at 214.63 133.35 0) (unit 1)
     (in_bom yes) (on_board yes)
     (property "Reference" "#PWR021" (id 0) (at 214.63 139.7 0)
@@
     (pin "1")
   )
-  (symbol (lib_id "Device:Q_NPN_BEC") (at 212.09 125.73 0)
+  (symbol (lib_id "Device:Q_NPN_BEC") (at 212.09 125.73 0) (unit 1)
     (in_bom yes) (on_board yes)
     (property "Reference" "Q2" (id 0) (at 216.9414 124.5616 0)
@@
     (pin "2")
   )
-  (symbol (lib_id "Device:C") (at 41.91 72.39 0) (mirror y)
+  (symbol (lib_id "Device:C") (at 41.91 72.39 0) (mirror y) (unit 1)
     (in_bom yes) (on_board yes)
     (property "Reference" "C4" (id 0) (at 44.45 69.85 0)
@@
     (pin "1")
   )
-  (symbol (lib_id "Device:C") (at 48.26 72.39 0)
+  (symbol (lib_id "Device:C") (at 48.26 72.39 0) (unit 1)
     (in_bom yes) (on_board yes)
     (property "Reference" "C5" (id 0) (at 48.26 69.85 0)
@@
     (pin "2")
   )
-  (symbol (lib_id "Device:C") (at 54.61 72.39 0)
+  (symbol (lib_id "Device:C") (at 54.61 72.39 0) (unit 1)
     (in_bom yes) (on_board yes)
     (property "Reference" "C7" (id 0) (at 54.61 69.85 0)
@@
     (pin "2")
   )
-  (symbol (lib_id "Device:C") (at 60.96 72.39 0)
+  (symbol (lib_id "Device:C") (at 60.96 72.39 0) (unit 1)
     (in_bom yes) (on_board yes)
     (property "Reference" "C8" (id 0) (at 60.96 69.85 0)
@@
     (pin "2")
   )
-  (symbol (lib_id "Device:C") (at 67.31 72.39 0)
+  (symbol (lib_id "Device:C") (at 67.31 72.39 0) (unit 1)
     (in_bom yes) (on_board yes)
     (property "Reference" "C9" (id 0) (at 67.31 69.85 0)
@@
     (pin "2")
   )
-  (symbol (lib_id "Device:R") (at 43.18 86.36 0)
+  (symbol (lib_id "Device:R") (at 43.18 86.36 0) (unit 1)
     (in_bom yes) (on_board yes)
     (property "Reference" "R3" (id 0) (at 39.37 86.36 0))
@@
     (pin "2")
   )
-  (symbol (lib_id "Device:R") (at 22.86 97.79 90)
+  (symbol (lib_id "Device:R") (at 22.86 97.79 90) (unit 1)
     (in_bom yes) (on_board yes)
     (property "Reference" "R1" (id 0) (at 22.86 95.25 90))
@@
     (pin "1")
   )
-  (symbol (lib_id "Device:R") (at 91.44 149.86 0)
+  (symbol (lib_id "Device:R") (at 91.44 149.86 0) (unit 1)
     (in_bom yes) (on_board yes)
     (property "Reference" "R5" (id 0) (at 93.98 149.86 0))
@@
     (pin "2")
   )
-  (symbol (lib_id "Device:R") (at 96.52 149.86 0)
+  (symbol (lib_id "Device:R") (at 96.52 149.86 0) (unit 1)
     (in_bom yes) (on_board yes)
     (property "Reference" "R6" (id 0) (at 99.06 149.86 0))
@@
     (pin "1")
   )
-  (symbol (lib_id "Device:C") (at 121.92 176.53 0)
+  (symbol (lib_id "Device:C") (at 121.92 176.53 0) (unit 1)
     (in_bom yes) (on_board yes)
     (property "Reference" "C14" (id 0) (at 121.92 173.99 0)
@@
     (pin "1")
   )
-  (symbol (lib_id "Device:C") (at 30.48 72.39 0)
+  (symbol (lib_id "Device:C") (at 30.48 72.39 0) (unit 1)
     (in_bom yes) (on_board yes)
     (property "Reference" "C3" (id 0) (at 30.48 69.85 0)
